Commit message: Camera plugin + topic

File: wcr_description/urdf/wcr_base.xacro (robot description, xacro)
@@ -29,5 +29,5 @@
             <origin xyz="0 0 0" rpy="0 0 0"/>
             <mass value="0.05"/>
-            <inertia ixx="1e-5" ixy="0" ixz="0" iyy="1e-5" iyz="0" izz="1e-5"/>
+            <!-- inertia ixx="1e-5" ixy="0" ixz="0" iyy="1e-5" iyz="0" izz="1e-5"/ -->
         </inertial>
     </link>

Commit message: Barometer + Distance measurement sensors

File: wcr_description/urdf/wcr_base.xacro (robot description, xacro)
@@ -32,4 +32,12 @@
         </inertial>
     </link>
+    <!-- BAROMETER LINK -->
+    <joint name="barometer_joint" type="fixed">
+        <parent link="chassis_link"/>
+        <child link="barometer_link"/>
+        <origin xyz="0.06 0 0.1"/>
+    </joint>
+    <link name="barometer_link">
+    </link>
     <!-- T265 LINK -->
     <joint name="camera_joint" type="fixed">
@@ -55,4 +63,12 @@
     </joint>
     <link name="marvelmind_link">
+    </link>
+    <!-- DISTANCE SENSOR LINK -->
+    <joint name="distance_sensor_joint" type="fixed">
+        <parent link="chassis_link"/>
+        <child link="distance_sensor_link"/>
+        <origin xyz="0.16 0.0 0.05" rpy="0 ${pi/2} 0"/>
+    </joint>
+    <link name="distance_sensor_link">
     </link>
     <!-- CHASSIS LINK-->

Commit message: Latest

File: wcr_description/urdf/wcr_base.xacro (robot description, xacro)
@@ -23,5 +23,5 @@
         <parent link="chassis_link"/>
         <child link="imu_link"/>
-        <origin xyz="0.06551 0 0.098"/>
+        <origin xyz="${imu_x} ${imu_y} ${imu_z}" rpy="${imu_roll} ${imu_pitch} ${imu_yaw}"/>
     </joint>
     <link name="imu_link">
@@ -36,5 +36,5 @@
         <parent link="chassis_link"/>
         <child link="barometer_link"/>
-        <origin xyz="0.06 0 0.1"/>
+        <origin xyz="${barometer_x} ${barometer_y} ${barometer_z}" rpy="${barometer_roll} ${barometer_pitch} ${barometer_yaw}"/>
     </joint>
     <link name="barometer_link">
@@ -44,7 +44,15 @@
         <parent link="chassis_link"/>
         <child link="t265_link"/>
-        <origin xyz="0.14885 0.00922 0.06659"/>
+        <origin xyz="${camera_x} ${camera_y} ${camera_z}" rpy="${camera_roll} ${camera_pitch} ${camera_yaw}"/>
     </joint>
     <link name="t265_link">
+    </link>
+    <!-- OPTICAL FLOW LINK -->
+    <joint name="optical_flow_joint" type="fixed">
+        <parent link="chassis_link"/>
+        <child link="optical_flow_link"/>
+        <origin xyz="${optical_flow_x} ${optical_flow_y} ${optical_flow_z}" rpy="${optical_flow_roll} ${optical_flow_pitch} ${optical_flow_yaw}"/>
+    </joint>
+    <link name="optical_flow_link">
     </link>
     <!-- T265 ODOM -->
@@ -52,5 +60,5 @@
         <parent link="chassis_link"/>
         <child link="t265_odom_frame"/>
-        <origin xyz="0.14885 0.00922 0.06659"/>
+        <origin xyz="${camera_x} ${camera_y} ${camera_z}" rpy="${camera_roll} ${camera_pitch} ${camera_yaw}"/>
     </joint>
     <link name="t265_odom_frame">
@@ -68,5 +76,5 @@
         <parent link="chassis_link"/>
         <child link="distance_sensor_link"/>
-        <origin xyz="0.16 0.0 0.05" rpy="0 ${pi/2} 0"/>
+        <origin xyz="${distance_sensor_x} ${distance_sensor_y} ${distance_sensor_z}" rpy="${distance_sensor_roll} ${distance_sensor_pitch} ${distance_sensor_yaw}"/>
     </joint>
     <link name="distance_sensor_link">

File: wcr_description/urdf/wcr_params.xacro (robot description, xacro)
@@ -15,4 +15,66 @@
     <xacro:arg name="chassis_mass" default="3.0"/>
     <xacro:arg name="chassis_inertia" default="0.003"/>
+    <!-- Sensor Mount Poses -->
+    <xacro:arg name="imu_x" default="0.06551"/>
+    <xacro:arg name="imu_y" default="0.0"/>
+    <xacro:arg name="imu_z" default="0.098"/>
+    <xacro:arg name="imu_roll" default="0.0"/>
+    <xacro:arg name="imu_pitch" default="0.0"/>
+    <xacro:arg name="imu_yaw" default="0.0"/>
+    <xacro:arg name="camera_x" default="0.14885"/>
+    <xacro:arg name="camera_y" default="0.00922"/>
+    <xacro:arg name="camera_z" default="0.06659"/>
+    <xacro:arg name="camera_roll" default="0.0"/>
+    <xacro:arg name="camera_pitch" default="0.0"/>
+    <xacro:arg name="camera_yaw" default="0.0"/>
+    <xacro:arg name="optical_flow_x" default="0.06"/>
+    <xacro:arg name="optical_flow_y" default="0.0"/>
+    <xacro:arg name="optical_flow_z" default="0.095"/>
+    <xacro:arg name="optical_flow_roll" default="0.0"/>
+    <xacro:arg name="optical_flow_pitch" default="-1.57079632679"/>
+    <xacro:arg name="optical_flow_yaw" default="0.0"/>
+    <xacro:arg name="barometer_x" default="0.06"/>
+    <xacro:arg name="barometer_y" default="0.0"/>
+    <xacro:arg name="barometer_z" default="0.1"/>
+    <xacro:arg name="barometer_roll" default="0.0"/>
+    <xacro:arg name="barometer_pitch" default="0.0"/>
+    <xacro:arg name="barometer_yaw" default="0.0"/>
+    <xacro:arg name="distance_sensor_x" default="0.16"/>
+    <xacro:arg name="distance_sensor_y" default="0.0"/>
+    <xacro:arg name="distance_sensor_z" default="0.05"/>
+    <xacro:arg name="distance_sensor_roll" default="0.0"/>
+    <xacro:arg name="distance_sensor_pitch" default="1.57079632679"/>
+    <xacro:arg name="distance_sensor_yaw" default="0.0"/>
+    <!-- Sensor Rates -->
+    <xacro:arg name="imu_rate_hz" default="100.0"/>
+    <xacro:arg name="camera_rate_hz" default="30.0"/>
+    <xacro:arg name="optical_flow_rate_hz" default="50.0"/>
+    <xacro:arg name="barometer_rate_hz" default="25.0"/>
+    <xacro:arg name="distance_rate_hz" default="20.0"/>
+    <!-- Sensor Noise -->
+    <xacro:arg name="imu_gyro_stddev" default="0.001"/>
+    <xacro:arg name="imu_accel_stddev" default="0.01"/>
+    <xacro:arg name="camera_noise_stddev" default="0.0005"/>
+    <xacro:arg name="optical_flow_noise_stddev" default="0.0005"/>
+    <xacro:arg name="barometer_noise_stddev" default="10.0"/>
+    <xacro:arg name="distance_noise_stddev" default="0.0005"/>
+    <!-- Camera / Optical Flow -->
+    <xacro:arg name="camera_width" default="800"/>
+    <xacro:arg name="camera_height" default="800"/>
+    <xacro:arg name="camera_hfov" default="1.3962634"/>
+    <xacro:arg name="optical_flow_width" default="320"/>
+    <xacro:arg name="optical_flow_height" default="240"/>
+    <xacro:arg name="optical_flow_hfov" default="1.3962634"/>
+    <!-- Distance Sensor -->
+    <xacro:arg name="distance_min_m" default="0.05"/>
+    <xacro:arg name="distance_max_m" default="5.0"/>
+    <xacro:arg name="distance_resolution_m" default="0.01"/>
+    <!-- Barometer -->
+    <xacro:arg name="barometer_reference_altitude" default="0.0"/>
+    <!-- Thruster / Environment -->
+    <xacro:arg name="air_density" default="1.225"/>
+    <xacro:arg name="thruster_coefficient" default="0.1"/>
+    <xacro:arg name="propeller_diameter_main" default="0.2286"/>
+    <xacro:arg name="propeller_diameter_edf" default="0.11"/>
     <!-- Steering -->
     <xacro:arg name="steering_height" default="0.05029"/>
@@ -55,4 +117,61 @@
     <xacro:property name="chassis_mass" value="$(arg chassis_mass)"/>
     <xacro:property name="chassis_inertia" value="$(arg chassis_inertia)"/>
+    <!-- SENSOR MOUNT POSE PARAMETERS -->
+    <xacro:property name="imu_x" value="$(arg imu_x)"/>
+    <xacro:property name="imu_y" value="$(arg imu_y)"/>
+    <xacro:property name="imu_z" value="$(arg imu_z)"/>
+    <xacro:property name="imu_roll" value="$(arg imu_roll)"/>
+    <xacro:property name="imu_pitch" value="$(arg imu_pitch)"/>
+    <xacro:property name="imu_yaw" value="$(arg imu_yaw)"/>
+    <xacro:property name="camera_x" value="$(arg camera_x)"/>
+    <xacro:property name="camera_y" value="$(arg camera_y)"/>
+    <xacro:property name="camera_z" value="$(arg camera_z)"/>
+    <xacro:property name="camera_roll" value="$(arg camera_roll)"/>
+    <xacro:property name="camera_pitch" value="$(arg camera_pitch)"/>
+    <xacro:property name="camera_yaw" value="$(arg camera_yaw)"/>
+    <xacro:property name="optical_flow_x" value="$(arg optical_flow_x)"/>
+    <xacro:property name="optical_flow_y" value="$(arg optical_flow_y)"/>
+    <xacro:property name="optical_flow_z" value="$(arg optical_flow_z)"/>
+    <xacro:property name="optical_flow_roll" value="$(arg optical_flow_roll)"/>
+    <xacro:property name="optical_flow_pitch" value="$(arg optical_flow_pitch)"/>
+    <xacro:property name="optical_flow_yaw" value="$(arg optical_flow_yaw)"/>
+    <xacro:property name="barometer_x" value="$(arg barometer_x)"/>
+    <xacro:property name="barometer_y" value="$(arg barometer_y)"/>
+    <xacro:property name="barometer_z" value="$(arg barometer_z)"/>
+    <xacro:property name="barometer_roll" value="$(arg barometer_roll)"/>
+    <xacro:property name="barometer_pitch" value="$(arg barometer_pitch)"/>
+    <xacro:property name="barometer_yaw" value="$(arg barometer_yaw)"/>
+    <xacro:property name="distance_sensor_x" value="$(arg distance_sensor_x)"/>
+    <xacro:property name="distance_sensor_y" value="$(arg distance_sensor_y)"/>
+    <xacro:property name="distance_sensor_z" value="$(arg distance_sensor_z)"/>
+    <xacro:property name="distance_sensor_roll" value="$(arg distance_sensor_roll)"/>
+    <xacro:property name="distance_sensor_pitch" value="$(arg distance_sensor_pitch)"/>
+    <xacro:property name="distance_sensor_yaw" value="$(arg distance_sensor_yaw)"/>
+    <!-- SENSOR CONFIG PARAMETERS -->
+    <xacro:property name="imu_rate_hz" value="$(arg imu_rate_hz)"/>
+    <xacro:property name="camera_rate_hz" value="$(arg camera_rate_hz)"/>
+    <xacro:property name="optical_flow_rate_hz" value="$(arg optical_flow_rate_hz)"/>
+    <xacro:property name="barometer_rate_hz" value="$(arg barometer_rate_hz)"/>
+    <xacro:property name="distance_rate_hz" value="$(arg distance_rate_hz)"/>
+    <xacro:property name="imu_gyro_stddev" value="$(arg imu_gyro_stddev)"/>
+    <xacro:property name="imu_accel_stddev" value="$(arg imu_accel_stddev)"/>
+    <xacro:property name="camera_noise_stddev" value="$(arg camera_noise_stddev)"/>
+    <xacro:property name="optical_flow_noise_stddev" value="$(arg optical_flow_noise_stddev)"/>
+    <xacro:property name="barometer_noise_stddev" value="$(arg barometer_noise_stddev)"/>
+    <xacro:property name="distance_noise_stddev" value="$(arg distance_noise_stddev)"/>
+    <xacro:property name="camera_width" value="$(arg camera_width)"/>
+    <xacro:property name="camera_height" value="$(arg camera_height)"/>
+    <xacro:property name="camera_hfov" value="$(arg camera_hfov)"/>
+    <xacro:property name="optical_flow_width" value="$(arg optical_flow_width)"/>
+    <xacro:property name="optical_flow_height" value="$(arg optical_flow_height)"/>
+    <xacro:property name="optical_flow_hfov" value="$(arg optical_flow_hfov)"/>
+    <xacro:property name="distance_min_m" value="$(arg distance_min_m)"/>
+    <xacro:property name="distance_max_m" value="$(arg distance_max_m)"/>
+    <xacro:property name="distance_resolution_m" value="$(arg distance_resolution_m)"/>
+    <xacro:property name="barometer_reference_altitude" value="$(arg barometer_reference_altitude)"/>
+    <xacro:property name="air_density" value="$(arg air_density)"/>
+    <xacro:property name="thruster_coefficient" value="$(arg thruster_coefficient)"/>
+    <xacro:property name="propeller_diameter_main" value="$(arg propeller_diameter_main)"/>
+    <xacro:property name="propeller_diameter_edf" value="$(arg propeller_diameter_edf)"/>
     <!-- STEERING PARAMETERS -->
 	<xacro:property name="steering_height" value="$(arg steering_height)" />
